Commit message: add inertial

File: chapter3_ws/src/robot_description/urdf/robot_base.urdf.xacro (robot description, xacro)
@@ -3,4 +3,15 @@
 <xacro:include filename="$(find robot_description)/urdf/robot_essentials.xacro" />
 	<link name="base_link">
+		<inertial>
+			<origin xyz="0.0030946 4.78250032638821E-11 0.053305" rpy="0 0 0" />
+			<mass value="47.873" />
+			<inertia
+				ixx="0.774276574699151"
+				ixy="-1.03781944357671E-10"
+				ixz="0.00763014265820928"
+				iyy="1.64933255189991"
+				iyz="1.09578155845563E-12"
+				izz="2.1239326987473" />
+		</inertial>
 		<visual>
 			<origin xyz="0 0 0" rpy="1.5707963267949 0 3.14" />
@@ -8,4 +19,10 @@
 				<mesh filename="package://robot_description/meshes/robot_base.stl"/>
 			</geometry>
+		<collision>
+			<origin xyz="0 0 0" rpy="1.5707963267949 0 3.14" />
+			<geometry>
+				<mesh filename="package://robot_description/meshes/robot_base.stl"/>
+			</geometry>
+		</collision>
 			<material name="">
 				<color rgba="0.79216 0.81961 0.93333 1" />

File: chapter3_ws/src/robot_description/urdf/robot_essentials.xacro (robot description, xacro)
@@ -3,4 +3,15 @@
 <xacro:macro name="robot_wheel" params="prefix">
 	<link name="${prefix}_wheel">
+		<inertial>
+			<origin xyz="-4.1867E-18 0.0068085 -1.65658661799998E-18" rpy="0 0 0" />
+			<mass value="2.6578" />
+			<inertia
+				ixx="0.00856502765719703"
+				ixy="1.5074118157338E-19"
+				ixz="-4.78150098725052E-19"
+				iyy="0.0136064032096"
+				iyz="-2.68136447099727E-19"
+				izz="0.00856502765719703" />
+		</inertial>
 		<visual>
 			<origin xyz="0 0 0" rpy="1.5707963267949 0 0" />
@@ -8,4 +19,10 @@
 					<mesh filename="package://robot_description/meshes/wheel.stl"/>
 				</geometry>
+		<collision>
+			<origin xyz="0 0 0" rpy="1.5707963267949 0 0" />
+				<geometry>
+					<mesh filename="package://robot_description/meshes/wheel.stl"/>
+				</geometry>
+		</collision>
 				<material name="">
 					<color rgba="0.79216 0.81961 0.93333 1" />

Commit message: fix <collision> in 2 files

File: chapter3_ws/src/robot_description/urdf/robot_base.urdf.xacro (robot description, xacro)
@@ -21,4 +21,8 @@
 				<mesh filename="package://robot_description/meshes/robot_base.stl"/>
 			</geometry>
+			<material name="">
+				<color rgba="0.79216 0.81961 0.93333 1" />
+			</material>
+		</visual>
 		<collision>
 			<origin xyz="0 0 0" rpy="1.5707963267949 0 3.14" />
@@ -27,8 +31,4 @@
 			</geometry>
 		</collision>
-			<material name="">
-				<color rgba="0.79216 0.81961 0.93333 1" />
-			</material>
-		</visual>
 	</link>
 <xacro:robot_wheel prefix="front_left"/>

File: chapter3_ws/src/robot_description/urdf/robot_essentials.xacro (robot description, xacro)
@@ -19,4 +19,8 @@
 					<mesh filename="package://robot_description/meshes/wheel.stl"/>
 				</geometry>
+				<material name="">
+					<color rgba="0.79216 0.81961 0.93333 1" />
+				</material>
+		</visual>
 		<collision>
 			<origin xyz="0 0 0" rpy="1.5707963267949 0 0" />
@@ -25,8 +29,4 @@
 				</geometry>
 		</collision>
-				<material name="">
-					<color rgba="0.79216 0.81961 0.93333 1" />
-				</material>
-		</visual>
 	</link>
 </xacro:macro>
